Commit message: project reumes

File: install/drone_description/share/drone_description/urdf/common_properties.xacro (robot description, xacro)
@@ -1,48 +1 @@
-<?xml version="1.0"?>
-<robot xmlns:xacro="http://www.ros.org/wiki/xacro">
-    <material name="green">
-        <color rgba="0 0 1 1" />
-    </material>
-    <material name="grey">
-        <color rgba="1 1 1 1" />
-    </material>
-    <material name="blue">
-        <color rgba="0 0 1 1" />
-    </material>
-    <material name="black">
-        <color rgba="0 0 0 1" />
-    </material>
-    <material name="yellow">
-        <color rgba="1 1 0 1" />
-    </material>
-    <material name="red">
-        <color rgba="1 0 0 1" />
-    </material>
-    <xacro:macro name="box_inertia" params="m x y z o_xyz o_rpy">
-        <inertial>
-            <mass value="${m}" />
-            <origin xyz="${o_xyz}" rpy="${o_rpy}" />
-            <inertia ixx="${(m/12)*(y*y + z*z)}" ixy="0" ixz="0"
-                     iyy="${(m/12)*(x*x + z*z)}" iyz="0"
-                     izz="${(m/12)*(x*x + y*y)}" />
-        </inertial>
-    </xacro:macro>
-    <xacro:macro name="cylinder_inertia" params="m r l o_xyz o_rpy">
-        <inertial>
-            <mass value="${m}" />
-            <origin xyz="${o_xyz}" rpy="${o_rpy}" />
-            <inertia ixx="${(m/12)*(3*r*r + l*l)}" ixy="0" ixz="0"
-                     iyy="${(m/12)*(3*r*r + l*l)}" iyz="0"
-                     izz="${(m/2)*(r*r)}" />
-        </inertial>
-    </xacro:macro>
-    <xacro:macro name="sphere_inertia" params="m r o_xyz o_rpy">
-        <inertial>
-            <mass value="${m}" />
-            <origin xyz="${o_xyz}" rpy="${o_rpy}" />
-            <inertia ixx="${(2*m/5)*(r*r)}" ixy="0" ixz="0"
-                     iyy="${(2*m/5)*(r*r)}" iyz="0"
-                     izz="${(2*m/5)*(r*r)}" />
-        </inertial>
-    </xacro:macro>
-</robot>
+/home/galdrux/gazebo_projects/drone_ws/src/drone_description/urdf/common_properties.xacro

File: install/drone_description/share/drone_description/urdf/drone.urdf.xacro (robot description, xacro)
@@ -1,380 +1 @@
-<?xml version="1.0"?>
-<robot name="drone" xmlns:xacro="http://www.ros.org/wiki/xacro">
-  <xacro:include filename="common_properties.xacro" />
-  <xacro:include filename="drone_gazebo.xacro" />
-  <xacro:include filename="imu_sensor.xacro" />
-  <xacro:property name="base_length" value="0.15" />
-  <xacro:property name="base_width" value="0.15" />
-  <xacro:property name="base_height" value="0.05" />
-  <xacro:property name="arm_length" value="0.15" />
-  <xacro:property name="arm_width" value="0.015" />
-  <xacro:property name="arm_height" value="0.015" />
-  <xacro:property name="shaft_radius" value="0.002" />
-  <xacro:property name="shaft_length" value="0.02" />
-  <xacro:property name="propeller_radius" value="0.06" />
-  <xacro:property name="propeller_length" value="0.004" />
-  <xacro:property name="stand_radius" value="0.01" />
-  <xacro:property name="stand_length" value="0.1" />
-  <link name="base_footprint" />
-  <link name="base_link">
-    <visual>
-      <geometry>
-        <box size="${base_length} ${base_width} ${base_height}"/>
-      </geometry>
-      <origin xyz="0 0 0" rpy="0 0 0"/>
-      <material name="black"/>
-    </visual>
-    <collision>
-      <geometry>
-        <box size="${base_length} ${base_width} ${base_height}"/>
-      </geometry>
-      <origin xyz="0 0 0" rpy="0 0 0"/>
-    </collision>
-    <xacro:box_inertia m="0.3" x="${base_length}" y="${base_width}" z="${base_height}" o_xyz="0 0 0" o_rpy="0 0 0" />
-  </link>
-  <link name="front_right_arm_link" >
-    <visual>
-      <geometry>
-        <box size="${arm_length} ${arm_width} ${arm_height}" />
-      </geometry>
-      <origin xyz="${arm_length/2.0} 0 0" rpy="0 0 0" />
-      <material name="blue"/>
-    </visual>
-    <collision>
-      <geometry>
-        <box size="${arm_length} ${arm_width} ${arm_height}" />
-      </geometry>
-      <origin xyz="${arm_length/2.0} 0 0" rpy="0 0 0" />
-    </collision>
-    <xacro:box_inertia m="0.025" x="${arm_length}" y="${arm_width}" z="${arm_height}" o_xyz="${arm_length/2.0} 0 0" o_rpy="0 0 0" />
-  </link>
-  <link name="front_left_arm_link" >
-    <visual>
-      <geometry>
-        <box size="${arm_length} ${arm_width} ${arm_height}" />
-      </geometry>
-      <origin xyz="${arm_length/2.0} 0 0" rpy="0 0 0" />
-      <material name="blue"/>
-    </visual>
-    <collision>
-      <geometry>
-        <box size="${arm_length} ${arm_width} ${arm_height}" />
-      </geometry>
-      <origin xyz="${arm_length/2.0} 0 0" rpy="0 0 0" />
-    </collision>
-    <xacro:box_inertia m="0.025" x="${arm_length}" y="${arm_width}" z="${arm_height}" o_xyz="${arm_length/2.0} 0 0" o_rpy="0 0 0" />
-  </link>
-  <link name="back_right_arm_link" >
-    <visual>
-      <geometry>
-        <box size="${arm_length} ${arm_width} ${arm_height}" />
-      </geometry>
-      <origin xyz="${arm_length/2.0} 0 0" rpy="0 0 0" />
-      <material name="blue"/>
-    </visual>
-    <collision>
-      <geometry>
-        <box size="${arm_length} ${arm_width} ${arm_height}" />
-      </geometry>
-      <origin xyz="${arm_length/2.0} 0 0" rpy="0 0 0" />
-    </collision>
-    <xacro:box_inertia m="0.025" x="${arm_length}" y="${arm_width}" z="${arm_height}" o_xyz="${arm_length/2.0} 0 0" o_rpy="0 0 0" />
-  </link>
-  <link name="back_left_arm_link" >
-    <visual>
-      <geometry>
-        <box size="${arm_length} ${arm_width} ${arm_height}" />
-      </geometry>
-      <origin xyz="${arm_length/2.0} 0 0" rpy="0 0 0" />
-      <material name="blue"/>
-    </visual>
-    <collision>
-      <geometry>
-        <box size="${arm_length} ${arm_width} ${arm_height}" />
-      </geometry>
-      <origin xyz="${arm_length/2.0} 0 0" rpy="0 0 0" />
-    </collision>
-    <xacro:box_inertia m="0.025" x="${arm_length}" y="${arm_width}" z="${arm_height}" o_xyz="${arm_length/2.0} 0 0" o_rpy="0 0 0" />
-  </link>
-  <link name="front_right_shaft_link" >
-    <visual>
-      <geometry>
-        <cylinder radius="${shaft_radius}" length="${shaft_length}" />
-      </geometry>
-      <origin xyz="0 0 ${shaft_length/2.0}" rpy="0 0 0" />
-      <material name="grey"/>
-    </visual>
-    <collision>
-      <geometry>
-        <cylinder radius="${shaft_radius}" length="${shaft_length}" />
-      </geometry>
-      <origin xyz="0 0 ${shaft_length/2.0}" rpy="0 0 0" />
-    </collision>
-    <xacro:cylinder_inertia m="0.03" r="${shaft_radius}" l="${shaft_length}" o_xyz="0 0 ${shaft_length/2.0}" o_rpy="0 0 0" />
-  </link>
-  <link name="front_left_shaft_link" >
-    <visual>
-      <geometry>
-        <cylinder radius="${shaft_radius}" length="${shaft_length}" />
-      </geometry>
-      <origin xyz="0 0 ${shaft_length/2.0}" rpy="0 0 0" />
-      <material name="grey"/>
-    </visual>
-    <collision>
-      <geometry>
-        <cylinder radius="${shaft_radius}" length="${shaft_length}" />
-      </geometry>
-      <origin xyz="0 0 ${shaft_length/2.0}" rpy="0 0 0" />
-    </collision>
-    <xacro:cylinder_inertia m="0.03" r="${shaft_radius}" l="${shaft_length}" o_xyz="0 0 ${shaft_length/2.0}" o_rpy="0 0 0" />
-  </link>
-  <link name="back_right_shaft_link" >
-    <visual>
-      <geometry>
-        <cylinder radius="${shaft_radius}" length="${shaft_length}" />
-      </geometry>
-      <origin xyz="0 0 ${shaft_length/2.0}" rpy="0 0 0" />
-      <material name="grey"/>
-    </visual>
-    <collision>
-      <geometry>
-        <cylinder radius="${shaft_radius}" length="${shaft_length}" />
-      </geometry>
-      <origin xyz="0 0 ${shaft_length/2.0}" rpy="0 0 0" />
-    </collision>
-    <xacro:cylinder_inertia m="0.03" r="${shaft_radius}" l="${shaft_length}" o_xyz="0 0 ${shaft_length/2.0}" o_rpy="0 0 0" />
-  </link>
-  <link name="back_left_shaft_link" >
-    <visual>
-      <geometry>
-        <cylinder radius="${shaft_radius}" length="${shaft_length}" />
-      </geometry>
-      <origin xyz="0 0 ${shaft_length/2.0}" rpy="0 0 0" />
-      <material name="grey"/>
-    </visual>
-    <collision>
-      <geometry>
-        <cylinder radius="${shaft_radius}" length="${shaft_length}" />
-      </geometry>
-      <origin xyz="0 0 ${shaft_length/2.0}" rpy="0 0 0" />
-    </collision>
-    <xacro:cylinder_inertia m="0.03" r="${shaft_radius}" l="${shaft_length}" o_xyz="0 0 ${shaft_length/2.0}" o_rpy="0 0 0" />
-  </link>
-  <link name="front_right_propeller_link" >
-    <visual>
-      <geometry>
-        <cylinder radius="${propeller_radius}" length="${propeller_length}" />
-      </geometry>
-      <origin xyz="0 0 0" rpy="0 0 0" />
-      <material name="red"/>
-    </visual>
-    <collision>
-      <geometry>
-        <cylinder radius="${propeller_radius}" length="${propeller_length}" />
-      </geometry>
-      <origin xyz="0 0 0" rpy="0 0 0" />
-    </collision>
-    <xacro:cylinder_inertia m="0.006" r="${propeller_radius}" l="${propeller_length}" o_xyz="0 0 0" o_rpy="0 0 0" />
-  </link>
-  <link name="front_left_propeller_link" >
-    <visual>
-      <geometry>
-        <cylinder radius="${propeller_radius}" length="${propeller_length}" />
-      </geometry>
-      <origin xyz="0 0 0" rpy="0 0 0" />
-      <material name="red"/>
-    </visual>
-    <collision>
-      <geometry>
-        <cylinder radius="${propeller_radius}" length="${propeller_length}" />
-      </geometry>
-      <origin xyz="0 0 0" rpy="0 0 0" />
-    </collision>
-    <xacro:cylinder_inertia m="0.006" r="${propeller_radius}" l="${propeller_length}" o_xyz="0 0 0" o_rpy="0 0 0" />
-  </link>
-  <link name="back_right_propeller_link" >
-    <visual>
-      <geometry>
-        <cylinder radius="${propeller_radius}" length="${propeller_length}" />
-      </geometry>
-      <origin xyz="0 0 0" rpy="0 0 0" />
-      <material name="red"/>
-    </visual>
-    <collision>
-      <geometry>
-        <cylinder radius="${propeller_radius}" length="${propeller_length}" />
-      </geometry>
-      <origin xyz="0 0 0" rpy="0 0 0" />
-    </collision>
-    <xacro:cylinder_inertia m="0.006" r="${propeller_radius}" l="${propeller_length}" o_xyz="0 0 0" o_rpy="0 0 0" />
-  </link>
-  <link name="back_left_propeller_link" >
-    <visual>
-      <geometry>
-        <cylinder radius="${propeller_radius}" length="${propeller_length}" />
-      </geometry>
-      <origin xyz="0 0 0" rpy="0 0 0" />
-      <material name="red"/>
-    </visual>
-    <collision>
-      <geometry>
-        <cylinder radius="${propeller_radius}" length="${propeller_length}" />
-      </geometry>
-      <origin xyz="0 0 0" rpy="0 0 0" />
-    </collision>
-    <xacro:cylinder_inertia m="0.006" r="${propeller_radius}" l="${propeller_length}" o_xyz="0 0 0" o_rpy="0 0 0" />
-  </link>
-  <link name="right_stand_link">
-    <visual>
-      <geometry>
-        <cylinder radius="${stand_radius}" length="${stand_length}" />
-      </geometry>
-      <origin xyz="0 0 ${-stand_length/2.0}" rpy="0 0 0" />
-      <material name="yellow" />
-    </visual>
-    <collision>
-      <geometry>
-        <cylinder radius="${stand_radius}" length="${stand_length}" />
-      </geometry>
-      <origin xyz="0 0 ${-stand_length/2.0}" rpy="0 0 0" />
-    </collision>
-    <xacro:cylinder_inertia m="0.015" r="${stand_radius}" l="${stand_length}" o_xyz="0 0 ${-stand_length/2.0}" o_rpy="0 0 0" />
-  </link>
-  <link name="left_stand_link">
-    <visual>
-      <geometry>
-        <cylinder radius="${stand_radius}" length="${stand_length}" />
-      </geometry>
-      <origin xyz="0 0 ${-stand_length/2.0}" rpy="0 0 0" />
-      <material name="yellow" />
-    </visual>
-    <collision>
-      <geometry>
-        <cylinder radius="${stand_radius}" length="${stand_length}" />
-      </geometry>
-      <origin xyz="0 0 ${-stand_length/2.0}" rpy="0 0 0" />
-    </collision>
-    <xacro:cylinder_inertia m="0.015" r="${stand_radius}" l="${stand_length}" o_xyz="0 0 ${-stand_length/2.0}" o_rpy="0 0 0" />
-  </link>
-  <link name="right_stand_base_link">
-    <visual>
-      <geometry>
-        <cylinder radius="${stand_radius}" length="${base_length}" />
-      </geometry>
-      <origin xyz="0 0 0" rpy="0 ${-pi/2.0} 0" />
-      <material name="black" />
-    </visual>
-    <collision>
-      <geometry>
-        <cylinder radius="${stand_radius}" length="${base_length}" />
-      </geometry>
-      <origin xyz="0 0 0" rpy="0 ${-pi/2.0} 0" />
-    </collision>
-    <xacro:cylinder_inertia m="0.01" r="${stand_radius}" l="${base_length}" o_xyz="0 0 0" o_rpy="0 ${-pi/2.0} 0" />
-  </link>
-  <link name="left_stand_base_link">
-    <visual>
-      <geometry>
-        <cylinder radius="${stand_radius}" length="${base_length}" />
-      </geometry>
-      <origin xyz="0 0 0" rpy="0 ${-pi/2.0} 0" />
-      <material name="black" />
-    </visual>
-    <collision>
-      <geometry>
-        <cylinder radius="${stand_radius}" length="${base_length}" />
-      </geometry>
-      <origin xyz="0 0 0" rpy="0 ${-pi/2.0} 0" />
-    </collision>
-    <xacro:cylinder_inertia m="0.01" r="${stand_radius}" l="${base_length}" o_xyz="0 0 0" o_rpy="0 ${-pi/2.0} 0" />
-  </link>
-  <joint name="base_joint" type="fixed">
-    <parent link="base_footprint" />
-    <child link="base_link" />
-    <origin xyz="0 0 ${(base_height/2.0)+(stand_length)+(stand_radius/2.0)}" rpy="0 0 0" />
-  </joint>
-  <joint name="base_front_right_arm_joint" type="fixed">
-    <parent link="base_link" />
-    <child link="front_right_arm_link" />
-    <origin xyz="${base_length/2.0} ${base_width/2.0} 0" rpy="0 0 ${pi/4.0}" />
-  </joint>
-  <joint name="base_front_left_arm_joint" type="fixed">
-    <parent link="base_link" />
-    <child link="front_left_arm_link" />
-    <origin xyz="${base_length/2.0} ${-base_width/2.0} 0" rpy="0 0 ${-pi/4.0}" />
-  </joint>
-  <joint name="base_back_right_arm_joint" type="fixed">
-    <parent link="base_link" />
-    <child link="back_right_arm_link" />
-    <origin xyz="${-base_length/2.0} ${base_width/2.0} 0" rpy="0 0 ${3.0*pi/4.0}" />
-  </joint>
-  <joint name="base_back_left_arm_joint" type="fixed">
-    <parent link="base_link" />
-    <child link="back_left_arm_link" />
-    <origin xyz="${-base_length/2.0} ${-base_width/2.0} 0" rpy="0 0 ${-3.0*pi/4.0}" />
-  </joint>
-  <joint name="front_right_arm_shaft_joint" type="fixed">
-    <parent link="front_right_arm_link" />
-    <child link="front_right_shaft_link" />
-    <origin xyz="${9*arm_length/10.0} 0 ${arm_height/2.0}" rpy="0 0 0" />
-  </joint>
-  <joint name="front_left_arm_shaft_joint" type="fixed">
-    <parent link="front_left_arm_link" />
-    <child link="front_left_shaft_link" />
-    <origin xyz="${9*arm_length/10.0} 0 ${arm_height/2.0}" rpy="0 0 0" />
-  </joint>
-  <joint name="back_right_arm_shaft_joint" type="fixed">
-    <parent link="back_right_arm_link" />
-    <child link="back_right_shaft_link" />
-    <origin xyz="${9*arm_length/10.0} 0 ${arm_height/2.0}" rpy="0 0 0" />
-  </joint>
-  <joint name="back_left_arm_shaft_joint" type="fixed">
-    <parent link="back_left_arm_link" />
-    <child link="back_left_shaft_link" />
-    <origin xyz="${9*arm_length/10.0} 0 ${arm_height/2.0}" rpy="0 0 0" />
-  </joint>
-  <joint name="front_right_shaft_propeller" type="continuous">
-    <parent link="front_right_shaft_link" />
-    <child link="front_right_propeller_link" />
-    <origin xyz="0 0 ${shaft_length}"  rpy="0 0 0" />
-    <axis xyz="0 0 1" />
-  </joint>
-  <joint name="front_left_shaft_propeller" type="continuous">
-    <parent link="front_left_shaft_link" />
-    <child link="front_left_propeller_link" />
-    <origin xyz="0 0 ${shaft_length}"  rpy="0 0 0" />
-    <axis xyz="0 0 -1" />
-  </joint>
-  <joint name="back_right_shaft_propeller" type="continuous">
-    <parent link="back_right_shaft_link" />
-    <child link="back_right_propeller_link" />
-    <origin xyz="0 0 ${shaft_length}"  rpy="0 0 0" />
-    <axis xyz="0 0 -1" />
-  </joint>
-  <joint name="back_left_shaft_propeller" type="continuous">
-    <parent link="back_left_shaft_link" />
-    <child link="back_left_propeller_link" />
-    <origin xyz="0 0 ${shaft_length}"  rpy="0 0 0" />
-    <axis xyz="0 0 1" />
-  </joint>
-  <joint name="base_right_stand_joint" type="fixed">
-    <parent link="base_link" />
-    <child link="right_stand_link" />
-    <origin xyz="0 ${-base_width/3.0} ${-base_height/2.0}" rpy="${-pi/12.0} 0 0" />
-  </joint>
-  <joint name="base_left_stand_joint" type="fixed">
-    <parent link="base_link" />
-    <child link="left_stand_link" />
-    <origin xyz="0 ${base_width/3.0} ${-base_height/2.0}" rpy="${pi/12.0} 0 0" />
-  </joint>
-  <joint name="right_stand_base_joint" type="fixed">
-    <parent link="right_stand_link" />
-    <child link="right_stand_base_link" />
-    <origin xyz="0 0 ${-stand_length}" rpy="0 0 0" />
-  </joint>
-  <joint name="left_stand_base_joint" type="fixed">
-    <parent link="left_stand_link" />
-    <child link="left_stand_base_link" />
-    <origin xyz="0 0 ${-stand_length}" rpy="0 0 0" />
-  </joint>
-</robot>
+/home/galdrux/gazebo_projects/drone_ws/src/drone_description/urdf/drone.urdf.xacro

File: install/drone_description/share/drone_description/urdf/drone_gazebo.xacro (robot description, xacro)
@@ -1,98 +1 @@
-<?xml version="1.0"?>
-<robot xmlns:xacro="http://www.ros.org/wiki/xacro">
-    <gazebo>
-        <plugin filename="gz-sim-multicopter-motor-model-system" name="gz::sim::systems::MulticopterMotorModel" >
-            <robotNamespace>drone</robotNamespace>
-            <jointName>front_right_shaft_propeller</jointName>
-            <linkName>front_right_propeller_link</linkName>
-            <turningDirection>ccw</turningDirection>
-            <timeConstantUp>0.0125</timeConstantUp>
-            <timeConstantDown>0.025</timeConstantDown>
-            <maxRotVelocity>800.0</maxRotVelocity>
-            <motorConstant>8.54858e-06</motorConstant>
-            <momentConstant>0.016</momentConstant>
-            <commandSubTopic>gazebo/command/motor_speed</commandSubTopic>
-            <actuator_number>0</actuator_number>
-            <rotorDragCoefficient>8.06428e-05</rotorDragCoefficient>
-            <rollingMomentCoefficient>1e-06</rollingMomentCoefficient>
-            <motorSpeedPubTopic>motor_speed/0</motorSpeedPubTopic>
-            <rotorVelocitySlowdownSim>10</rotorVelocitySlowdownSim>
-            <motorType>velocity</motorType>
-        </plugin>
-    </gazebo>
-    <gazebo>
-        <plugin filename="gz-sim-multicopter-motor-model-system" name="gz::sim::systems::MulticopterMotorModel" >
-            <robotNamespace>drone</robotNamespace>
-            <jointName>back_left_shaft_propeller</jointName>
-            <linkName>back_left_propeller_link</linkName>
-            <turningDirection>ccw</turningDirection>
-            <timeConstantUp>0.0125</timeConstantUp>
-            <timeConstantDown>0.025</timeConstantDown>
-            <maxRotVelocity>800.0</maxRotVelocity>
-            <motorConstant>8.54858e-06</motorConstant>
-            <momentConstant>0.016</momentConstant>
-            <commandSubTopic>gazebo/command/motor_speed</commandSubTopic>
-            <actuator_number>1</actuator_number>
-            <rotorDragCoefficient>8.06428e-05</rotorDragCoefficient>
-            <rollingMomentCoefficient>1e-06</rollingMomentCoefficient>
-            <motorSpeedPubTopic>motor_speed/1</motorSpeedPubTopic>
-            <rotorVelocitySlowdownSim>10</rotorVelocitySlowdownSim>
-            <motorType>velocity</motorType>
-        </plugin>
-    </gazebo>
-    <gazebo>
-        <plugin filename="gz-sim-multicopter-motor-model-system" name="gz::sim::systems::MulticopterMotorModel" >
-            <robotNamespace>drone</robotNamespace>
-            <jointName>front_left_shaft_propeller</jointName>
-            <linkName>front_left_propeller_link</linkName>
-            <turningDirection>cw</turningDirection>
-            <timeConstantUp>0.0125</timeConstantUp>
-            <timeConstantDown>0.025</timeConstantDown>
-            <maxRotVelocity>800.0</maxRotVelocity>
-            <motorConstant>8.54858e-06</motorConstant>
-            <momentConstant>0.016</momentConstant>
-            <commandSubTopic>gazebo/command/motor_speed</commandSubTopic>
-            <actuator_number>2</actuator_number>
-            <rotorDragCoefficient>8.06428e-05</rotorDragCoefficient>
-            <rollingMomentCoefficient>1e-06</rollingMomentCoefficient>
-            <motorSpeedPubTopic>motor_speed/2</motorSpeedPubTopic>
-            <rotorVelocitySlowdownSim>10</rotorVelocitySlowdownSim>
-            <motorType>velocity</motorType>
-        </plugin>
-    </gazebo>
-    <gazebo>
-        <plugin filename="gz-sim-multicopter-motor-model-system" name="gz::sim::systems::MulticopterMotorModel" >
-            <robotNamespace>drone</robotNamespace>
-            <jointName>back_right_shaft_propeller</jointName>
-            <linkName>back_right_propeller_link</linkName>
-            <turningDirection>cw</turningDirection>
-            <timeConstantUp>0.0125</timeConstantUp>
-            <timeConstantDown>0.025</timeConstantDown>
-            <maxRotVelocity>800.0</maxRotVelocity>
-            <motorConstant>8.54858e-06</motorConstant>
-            <momentConstant>0.016</momentConstant>
-            <commandSubTopic>gazebo/command/motor_speed</commandSubTopic>
-            <actuator_number>3</actuator_number>
-            <rotorDragCoefficient>8.06428e-05</rotorDragCoefficient>
-            <rollingMomentCoefficient>1e-06</rollingMomentCoefficient>
-            <motorSpeedPubTopic>motor_speed/3</motorSpeedPubTopic>
-            <rotorVelocitySlowdownSim>10</rotorVelocitySlowdownSim>
-            <motorType>velocity</motorType>
-        </plugin>
-    </gazebo>
-    <gazebo>
-        <plugin filename="gz-sim-odometry-publisher-system" name="gz::sim::systems::OdometryPublisher">
-            <dimensions>3</dimensions>
-            <odom_topic>odom</odom_topic>
-            <odom_publish_frequency>100</odom_publish_frequency>
-        </plugin>
-    </gazebo>
-    <gazebo>
-        <plugin filename="gz-sim-joint-state-publisher-system" name="gz::sim::systems::JointStatePublisher">
-            <joint_name>front_right_shaft_propeller</joint_name>
-            <joint_name>back_left_shaft_propeller</joint_name>
-            <joint_name>front_left_shaft_propeller</joint_name>
-            <joint_name>back_right_shaft_propeller</joint_name>
-        </plugin>
-    </gazebo>
-</robot>
+/home/galdrux/gazebo_projects/drone_ws/src/drone_description/urdf/drone_gazebo.xacro
